File: shield/kicad/Smartcard_Hat/Smartcard_Hat.kicad_sch (KiCad schematic)
At the start: 7 parts, among them J1 7712P0225A25LF, U6 ST8034HNQR

Commit message: add basic qr scanner
Parts:
- added C41: 1u, Capacitor_SMD:C_0805_2012Metric_Pad1.18x1.45mm_HandSolder, symbol Device:C
- added C42: 22u, Capacitor_SMD:C_0805_2012Metric_Pad1.18x1.45mm_HandSolder, symbol Device:C
- added J10: SFV12R-2STE1HLF, Library:AMPHENOL_SFV12R-2STE1HLF, symbol SFV12R-2STE1HLF:SFV12R-2STE1HLF
- added R48, R49, R50: 10k, Resistor_SMD:R_0402_1005Metric_Pad0.72x0.64mm_HandSolder, symbol Device:R_US
- added R51: 200R, Resistor_SMD:R_0402_1005Metric_Pad0.72x0.64mm_HandSolder, symbol Device:R_US
- renumbered J1 to J8
Connections:
- net +3V3: now also C41.1, C42.1, J10.2, R48.1, R49.1, R50.1
- net GND: now also C41.2, C42.2, J10.3
- net *3: no longer names the net of J12.5 (Pin_5)
- net *5: no longer names the net of J12.3 (Pin_3)
- net *6 renamed QR_UART_RX
- net QR_UART_RX: now also R51.1
- net 2: no longer names the net of J12.6 (Pin_6)
- net 4: no longer names the net of J12.4 (Pin_4)
- net 7 renamed QR_UART_TX
- net QR_UART_TX: now also J10.5, R49.2
- net RX/0: no longer names the net of J12.8 (Pin_8)
- net TX/1: no longer names the net of J12.7 (Pin_7)
- new net: J10.4, R50.2, R51.2
- new net QR_BEEP: J10.9
- new net QR_TRIG: J10.10, R48.2
- no-connect marks 3 -> 4
Other:
- moved on the sheet: J12

Commit message: re-org
Parts:
- removed C40, C42: 22u, Capacitor_SMD:C_0805_2012Metric_Pad1.18x1.45mm_HandSolder, symbol Device:C
- removed C41: 1u, Capacitor_SMD:C_0805_2012Metric_Pad1.18x1.45mm_HandSolder, symbol Device:C
- removed J10: SFV12R-2STE1HLF, Library:AMPHENOL_SFV12R-2STE1HLF, symbol SFV12R-2STE1HLF:SFV12R-2STE1HLF
- removed J11: ~, Connector_PinHeader_2.54mm:PinHeader_1x10_P2.54mm_Vertical_SMD_Pin1Left, symbol Connector_Generic:Conn_01x10
- removed J12, J9: ~, Connector_PinHeader_2.54mm:PinHeader_1x08_P2.54mm_Vertical_SMD_Pin1Left, symbol Connector_Generic:Conn_01x08
- removed J13: ~, Connector_PinHeader_2.54mm:PinHeader_1x06_P2.54mm_Vertical_SMD_Pin1Left, symbol Connector_Generic:Conn_01x06
- removed J8: 7712P0225A25LF, 7312P0225A13LF:AMPHENOL_7312P0225A13LF, symbol 7312P0225A13LF:7312P0225A13LF
- removed R48, R49, R50: 10k, Resistor_SMD:R_0402_1005Metric_Pad0.72x0.64mm_HandSolder, symbol Device:R_US
- removed R51: 200R, Resistor_SMD:R_0402_1005Metric_Pad0.72x0.64mm_HandSolder, symbol Device:R_US
- removed U6: ST8034HNQR, QFN24_4x4x0.8_STM, symbol specter_symbols:ST8034HNQR
Connections:
- no-connect marks 4 -> 0
Other:
- added sheet QR_Scanner (qr_scanner.kicad_sch)
- added sheet STM32F469I-DISCO-Interface (stm32f469i-disco-interface.kicad_sch)
- added sheet SmartCard_Reader (smartcard_reader.kicad_sch)
- note removed: "3V3"
- note removed: "5V"
- note removed: "GND"
- note removed: "IOREF"
- note removed: "NC"
- note removed: "NRST"
- note removed: "VIN"
