File: shield/kicad/Smartcard_Hat/smartcard_reader.kicad_sch (KiCad schematic)
At the start: 2 parts, among them J8 7712P0225A25LF, U1 ST8034HNQR

Commit message: wip
Parts:
- added C28, C29, C30, C31, C32, C33, C34, C36: u1, Capacitor_SMD:C_0805_2012Metric_Pad1.18x1.45mm_HandSolder, symbol Device:C
- added C35: 22u, Capacitor_SMD:C_0805_2012Metric_Pad1.18x1.45mm_HandSolder, symbol Device:C
- added C39: 1n, Capacitor_SMD:C_0805_2012Metric_Pad1.18x1.45mm_HandSolder, symbol Device:C
- added R31: 24k, Resistor_SMD:R_0402_1005Metric_Pad0.72x0.64mm_HandSolder, symbol Device:R_US
- added R32, R33, R34, R35, R43, R46, R47: 10k, Resistor_SMD:R_0402_1005Metric_Pad0.72x0.64mm_HandSolder, symbol Device:R_US
- added R36, R40, R41, R42, R44: 200R, Resistor_SMD:R_0402_1005Metric_Pad0.72x0.64mm_HandSolder, symbol Device:R_US
- added R45: 11.3k, Resistor_SMD:R_0402_1005Metric_Pad0.72x0.64mm_HandSolder, symbol Device:R_US
Connections:
- net +3V3: now also U1.1 (VDD(INTF)), C32.1, C33.1, C35.1, R31.1, R32.1, R33.1, R34.1, R35.1, R43.1
- net +5V: now also C34.1, C36.1
- net GND: now also C28.2, C29.2, C30.1, C31.1, C32.2, C33.2, C34.2, C35.2, C36.2, C39.2, R45.2, R46.2, R47.2
- net at J8.C1 (VCC), U1.15 (VCC): now also C28.1, C29.1, C30.2, C31.2
- net at U1.18 (PORADJ): now also C39.1, R43.2, R45.1
- net at U1.19 (*OFF): now also R31.2, R36.1
- net SC_VCC_SEL2: now reaches U1.2 (VCC_SEL2)
- net SC_VCC_SEL2: now also R33.2
- net at U1.20 (I/OUC): now also R40.2
- net at U1.21 (AUXUC1): now also R41.2
- net at U1.22 (AUXUC2): now also R42.2
- net at U1.23 (XTAL1): now also R44.2
- net SC_RST: now reaches U1.3 (RSTIN)
- net SC_RST: now also R47.1
- net SC_VCC_SEL1: now reaches U1.4 (VCC_SEL1)
- net SC_VCC_SEL1: now also R34.2
- net SC_nCMDVCC: now reaches U1.5 (*CMDVCC)
- net SC_nCMDVCC: now also R35.2
- net SC_CLKDIV1: now reaches U1.6 (CLKDIV1)
- net SC_CLKDIV1: now also R32.2
- net SC_CLKDIV2: now reaches U1.7 (CLKDIV2)
- net SC_CLKDIV2: now also R46.1
- new net SC_AUX1: R41.1
- new net SC_AUX2: R42.1
- new net SC_CLK: R44.1
- new net SC_IO: R40.1
- new net SC_nOFF: R36.2
- no-connect marks 1 -> 2

Commit message: wip
Parts:
- added R52: 10k, Resistor_SMD:R_0402_1005Metric_Pad0.72x0.64mm_HandSolder, symbol Device:R_US
- R44: value 200R -> 22R
Connections:
- net GND: now also R52.2
- net SC_nCMDVCC: now also R36.1; no longer R35.2, U1.5 (*CMDVCC)
- net SC_nOFF: now also R31.2, U1.19 (*OFF); no longer R36.2
- net at C30.2, C31.2, J8.C1 (VCC): no longer C28.1, C29.1, U1.15 (VCC)
- net at R44.2, U1.23 (XTAL1): now also R52.1
- net at J8.C2 (RST): no longer U1.14 (RST)
- net at J8.C3 (CLK): no longer U1.13 (CLK)
- net at J8.C4 (RFU): no longer U1.10 (AUX1)
- net at J8.C7 (I/O): no longer U1.9 (I/O)
- net at J8.C8 (RFU__1): no longer U1.11 (AUX2)
- net at J8.NO: no longer U1.8 (*PRES)
- new net: R35.2, R36.2, U1.5 (*CMDVCC)
Other:
- moved on the sheet: C28, C29, C39, R31, R33, R34, R35, R36, R40, R41, R42, R43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

Commit message: wip
Parts:
- renumbered U1 to U6
Connections:
- net GND: now also C30.2, C31.2; no longer C30.1, C31.1
- net at J8.C2 (RST): now also U6.14 (RST)
- net at J8.C3 (CLK): now also U6.13 (CLK)
- net at J8.C4 (RFU): now also U6.10 (AUX1)
- net at J8.C7 (I/O): now also U6.9 (I/O)
- net at J8.C8 (RFU__1): now also U6.11 (AUX2)
- net at J8.NO: now also U6.8 (*PRES)
- net at C29.1: now also C28.1, C30.1, C31.1, J8.C1 (VCC), U6.15 (VCC)
Other:
- moved on the sheet: C28, C29, C30, C31, C32, C33, C34, C35, C36, C39, J8, R31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

Commit message: wip
Parts:
- U6: footprint QFN24_4x4x0.8_STM -> Library:QFN24_4x4x0.8_STM
Connections:
- net SC_nCMDVCC: now also R35.2, U6.5 (*CMDVCC); no longer R36.1
- net SC_nOFF: now also R36.1; no longer R31.2, U6.19 (*OFF)
- new net: R31.2, R36.2, U6.19 (*OFF)
Other:
- moved on the sheet: R36
Changed lines of the file:
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@@
 	)
 	(junction
-		(at 104.14 86.36)
-		(diameter 0)
-		(color 0 0 0 0)
-	)
-	(junction
 		(at 71.12 93.98)
 		(diameter 0)
@@
 	)
 	(junction
-		(at 187.96 123.19)
+		(at 104.14 86.36)
 		(diameter 0)
 		(color 0 0 0 0)
 	)
 	(junction
-		(at 92.71 57.15)
+		(at 187.96 123.19)
 		(diameter 0)
 		(color 0 0 0 0)
 	)
 	(junction
-		(at 198.12 76.2)
+		(at 92.71 57.15)
 		(diameter 0)
 		(color 0 0 0 0)
 	)
 	(junction
-		(at 114.3 83.82)
+		(at 198.12 76.2)
 		(diameter 0)
 		(color 0 0 0 0)
@@
 	)
 	(junction
+		(at 114.3 83.82)
+		(diameter 0)
+		(color 0 0 0 0)
+	)
+	(junction
 		(at 133.35 45.72)
 		(diameter 0)
@@
 	(wire
 		(pts
-			(xy 53.34 86.36) (xy 104.14 86.36)
+			(xy 53.34 86.36) (xy 57.15 86.36)
 		)
 		(stroke
@@
 	(wire
 		(pts
+			(xy 53.34 83.82) (xy 114.3 83.82)
+		)
+		(stroke
+			(width 0)
+			(type default)
+		)
+	)
+	(wire
+		(pts
 			(xy 67.31 110.49) (xy 67.31 104.14)
 		)
@@
 	(wire
 		(pts
-			(xy 64.77 83.82) (xy 114.3 83.82)
+			(xy 182.88 68.58) (xy 182.88 83.82)
 		)
 		(stroke
@@
 	(wire
 		(pts
-			(xy 182.88 68.58) (xy 182.88 83.82)
+			(xy 64.77 86.36) (xy 104.14 86.36)
 		)
 		(stroke
@@
 	(wire
 		(pts
-			(xy 104.14 86.36) (xy 125.73 86.36)
-		)
-		(stroke
-			(width 0)
-			(type default)
-		)
-	)
-	(wire
-		(pts
 			(xy 220.98 93.98) (xy 215.9 93.98)
 		)
@@
 	(wire
 		(pts
+			(xy 104.14 86.36) (xy 125.73 86.36)
+		)
+		(stroke
+			(width 0)
+			(type default)
+		)
+	)
+	(wire
+		(pts
 			(xy 214.63 68.58) (xy 208.28 68.58)
 		)
@@
 	(wire
 		(pts
-			(xy 53.34 83.82) (xy 57.15 83.82)
-		)
-		(stroke
-			(width 0)
-			(type default)
-		)
-	)
-	(wire
-		(pts
 			(xy 81.28 57.15) (xy 81.28 60.96)
 		)
@@
 	(symbol
 		(lib_id "Device:R_US")
-		(at 60.96 83.82 90)
+		(at 60.96 86.36 90)
 		(unit 1)
 		(exclude_from_sim no)
@@
 		(fields_autoplaced yes)
 		(property "Reference" "R36"
-			(at 60.96 77.47 90)
+			(at 60.96 80.01 90)
 			(effects
 				(font
@@
 		)
 		(property "Value" "200R"
-			(at 60.96 80.01 90)
+			(at 60.96 82.55 90)
 			(effects
 				(font
@@
 		)
 		(property "Footprint" "Resistor_SMD:R_0402_1005Metric_Pad0.72x0.64mm_HandSolder"
-			(at 61.214 82.804 90)
+			(at 61.214 85.344 90)
 			(effects
 				(font
@@
 		)
 		(property "Datasheet" "~"
-			(at 60.96 83.82 0)
+			(at 60.96 86.36 0)
 			(effects
 				(font
@@
 		)
 		(property "Description" "Resistor, US symbol"
-			(at 60.96 83.82 0)
+			(at 60.96 86.36 0)
 			(effects
 				(font
@@
 			)
 		)
-		(property "Footprint" "QFN24_4x4x0.8_STM"
+		(property "Footprint" "Library:QFN24_4x4x0.8_STM"
 			(at 152.908 94.488 0)
 			(effects

Commit message: wip
Parts:
- added R1000, R1001: 0R, Resistor_SMD:R_0805_2012Metric_Pad1.20x1.40mm_HandSolder, symbol Device:R_US
- R31, R32, R33, R34, R35, R36, R40, R41, R42, R43, R44, R45, R46, R47, R52: footprint Resistor_SMD:R_0402_1005Metric_Pad0.72x0.64mm_HandSolder -> Resistor_SMD:R_0805_2012Metric_Pad1.20x1.40mm_HandSolder
Connections:
- net SC_RST: now also R1001.1; no longer U6.3 (RSTIN)
- net at U6.10 (AUX1): now also R1000.1; no longer J8.C4 (RFU)
- new net: J8.C4 (RFU), R1000.2
- new net: R1001.2, U6.3 (RSTIN)
Changed lines of the file:
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@@
 	)
 	(junction
-		(at 114.3 83.82)
+		(at 115.57 101.6)
 		(diameter 0)
 		(color 0 0 0 0)
 	)
 	(junction
-		(at 133.35 45.72)
+		(at 114.3 83.82)
 		(diameter 0)
 		(color 0 0 0 0)
 	)
 	(junction
-		(at 120.65 101.6)
+		(at 133.35 45.72)
 		(diameter 0)
 		(color 0 0 0 0)
@@
 	(wire
 		(pts
-			(xy 53.34 101.6) (xy 120.65 101.6)
+			(xy 53.34 101.6) (xy 115.57 101.6)
 		)
 		(stroke
@@
 	(wire
 		(pts
-			(xy 120.65 101.6) (xy 120.65 133.35)
+			(xy 115.57 101.6) (xy 115.57 133.35)
 		)
 		(stroke
@@
 	(wire
 		(pts
-			(xy 181.61 91.44) (xy 220.98 91.44)
+			(xy 181.61 91.44) (xy 210.82 91.44)
 		)
 		(stroke
@@
 	(wire
 		(pts
-			(xy 186.69 68.58) (xy 182.88 68.58)
+			(xy 115.57 133.35) (xy 120.65 133.35)
 		)
 		(stroke
@@
 	(wire
 		(pts
-			(xy 69.85 106.68) (xy 125.73 106.68)
+			(xy 186.69 68.58) (xy 182.88 68.58)
 		)
 		(stroke
@@
 	(wire
 		(pts
-			(xy 182.88 83.82) (xy 208.28 83.82)
+			(xy 69.85 106.68) (xy 125.73 106.68)
 		)
 		(stroke
@@
 	(wire
 		(pts
-			(xy 209.55 101.6) (xy 220.98 101.6)
+			(xy 182.88 83.82) (xy 208.28 83.82)
 		)
 		(stroke
@@
 	(wire
 		(pts
-			(xy 104.14 57.15) (xy 114.3 57.15)
+			(xy 209.55 101.6) (xy 220.98 101.6)
 		)
 		(stroke
@@
 	(wire
 		(pts
-			(xy 199.39 124.46) (xy 199.39 128.27)
+			(xy 104.14 57.15) (xy 114.3 57.15)
 		)
 		(stroke
@@
 	(wire
 		(pts
-			(xy 181.61 96.52) (xy 209.55 96.52)
+			(xy 199.39 124.46) (xy 199.39 128.27)
 		)
 		(stroke
@@
 	(wire
 		(pts
-			(xy 120.65 101.6) (xy 125.73 101.6)
+			(xy 181.61 96.52) (xy 209.55 96.52)
 		)
 		(stroke
@@
 	(wire
 		(pts
+			(xy 115.57 101.6) (xy 118.11 101.6)
+		)
+		(stroke
+			(width 0)
+			(type default)
+		)
+	)
+	(wire
+		(pts
 			(xy 187.96 128.27) (xy 187.96 124.46)
 		)
@@
 	(wire
 		(pts
+			(xy 218.44 91.44) (xy 220.98 91.44)
+		)
+		(stroke
+			(width 0)
+			(type default)
+		)
+	)
+	(wire
+		(pts
 			(xy 64.77 146.05) (xy 74.93 146.05)
 		)
@@
 	)
 	(symbol
+		(lib_id "Device:R_US")
+		(at 214.63 91.44 90)
+		(unit 1)
+		(exclude_from_sim no)
+		(in_bom yes)
+		(on_board yes)
+		(dnp no)
+		(fields_autoplaced yes)
+		(property "Reference" "R1000"
+			(at 214.63 85.09 90)
+			(effects
+				(font
+					(size 1.27 1.27)
+				)
+			)
+		)
+		(property "Value" "0R"
+			(at 214.63 87.63 90)
+			(effects
+				(font
+					(size 1.27 1.27)
+				)
+			)
+		)
+		(property "Footprint" "Resistor_SMD:R_0805_2012Metric_Pad1.20x1.40mm_HandSolder"
+			(at 214.884 90.424 90)
+			(effects
+				(font
+					(size 1.27 1.27)
+				)
+				(hide yes)
+			)
+		)
+		(property "Datasheet" "~"
+			(at 214.63 91.44 0)
+			(effects
+				(font
+					(size 1.27 1.27)
+				)
+				(hide yes)
+			)
+		)
+		(property "Description" "Resistor, US symbol"
+			(at 214.63 91.44 0)
+			(effects
+				(font
+					(size 1.27 1.27)
+				)
+				(hide yes)
+			)
+		)
+		(pin "1"
+		)
+		(pin "2"
+		)
+		(instances
+			(project "Smartcard_Hat"
+				(path "/e63e39d7-6ac0-4ffd-8aa3-1841a4541b55/b93ee573-e5a5-4e8b-bced-8a93bd527c9a"
+					(reference "R1000")
+					(unit 1)
+				)
+			)
+		)
+	)
+	(symbol
 		(lib_id "Device:C")
 		(at 224.79 72.39 0)
@@
 			)
 		)
-		(property "Footprint" "Resistor_SMD:R_0402_1005Metric_Pad0.72x0.64mm_HandSolder"
+		(property "Footprint" "Resistor_SMD:R_0805_2012Metric_Pad1.20x1.40mm_HandSolder"
 			(at 61.214 145.034 90)
 			(effects
@@
 			)
 		)
-		(property "Footprint" "Resistor_SMD:R_0402_1005Metric_Pad0.72x0.64mm_HandSolder"
+		(property "Footprint" "Resistor_SMD:R_0805_2012Metric_Pad1.20x1.40mm_HandSolder"
 			(at 72.136 65.024 90)
 			(effects
@@
 	)
 	(symbol
+		(lib_id "Device:R_US")
+		(at 121.92 101.6 90)
+		(unit 1)
+		(exclude_from_sim no)
+		(in_bom yes)
+		(on_board yes)
+		(dnp no)
+		(fields_autoplaced yes)
+		(property "Reference" "R1001"
+			(at 121.92 95.25 90)
+			(effects
+				(font
+					(size 1.27 1.27)
+				)
+			)
+		)
+		(property "Value" "0R"
+			(at 121.92 97.79 90)
+			(effects
+				(font
+					(size 1.27 1.27)
+				)
+			)
+		)
+		(property "Footprint" "Resistor_SMD:R_0805_2012Metric_Pad1.20x1.40mm_HandSolder"
+			(at 122.174 100.584 90)
+			(effects
+				(font
+					(size 1.27 1.27)
+				)
+				(hide yes)
+			)
+		)
+		(property "Datasheet" "~"
+			(at 121.92 101.6 0)
+			(effects
+				(font
+					(size 1.27 1.27)
+				)
+				(hide yes)
+			)
+		)
+		(property "Description" "Resistor, US symbol"
+			(at 121.92 101.6 0)
+			(effects
+				(font
+					(size 1.27 1.27)
+				)
+				(hide yes)
+			)
+		)
+		(pin "1"
+		)
+		(pin "2"
+		)
+		(instances
+			(project "Smartcard_Hat"
+				(path "/e63e39d7-6ac0-4ffd-8aa3-1841a4541b55/b93ee573-e5a5-4e8b-bced-8a93bd527c9a"
+					(reference "R1001")
+					(unit 1)
+				)
+			)
+		)
+	)
+	(symbol
 		(lib_name "GND_3")
 		(lib_id "power:GND")
@@
 			)
 		)
-		(property "Footprint" "Resistor_SMD:R_0402_1005Metric_Pad0.72x0.64mm_HandSolder"
+		(property "Footprint" "Resistor_SMD:R_0805_2012Metric_Pad1.20x1.40mm_HandSolder"
 			(at 61.214 109.474 90)
 			(effects
@@
 			)
 		)
-		(property "Footprint" "Resistor_SMD:R_0402_1005Metric_Pad0.72x0.64mm_HandSolder"
+		(property "Footprint" "Resistor_SMD:R_0805_2012Metric_Pad1.20x1.40mm_HandSolder"
 			(at 61.214 85.344 90)
 			(effects
@@
 			)
 		)
-		(property "Footprint" "Resistor_SMD:R_0402_1005Metric_Pad0.72x0.64mm_HandSolder"
+		(property "Footprint" "Resistor_SMD:R_0805_2012Metric_Pad1.20x1.40mm_HandSolder"
 			(at 188.976 132.334 90)
 			(effects
@@
 			)
 		)
-		(property "Footprint" "Resistor_SMD:R_0402_1005Metric_Pad0.72x0.64mm_HandSolder"
+		(property "Footprint" "Resistor_SMD:R_0805_2012Metric_Pad1.20x1.40mm_HandSolder"
 			(at 82.296 65.024 90)
 			(effects
@@
 			)
 		)
-		(property "Footprint" "Resistor_SMD:R_0402_1005Metric_Pad0.72x0.64mm_HandSolder"
+		(property "Footprint" "Resistor_SMD:R_0805_2012Metric_Pad1.20x1.40mm_HandSolder"
 			(at 115.316 65.024 90)
 			(effects
@@
 			)
 		)
-		(property "Footprint" "Resistor_SMD:R_0402_1005Metric_Pad0.72x0.64mm_HandSolder"
+		(property "Footprint" "Resistor_SMD:R_0805_2012Metric_Pad1.20x1.40mm_HandSolder"
 			(at 61.214 133.604 90)
 			(effects
@@
 			)
 		)
-		(property "Footprint" "Resistor_SMD:R_0402_1005Metric_Pad0.72x0.64mm_HandSolder"
+		(property "Footprint" "Resistor_SMD:R_0805_2012Metric_Pad1.20x1.40mm_HandSolder"
 			(at 110.236 137.414 90)
 			(effects
@@
 			)
 		)
-		(property "Footprint" "Resistor_SMD:R_0402_1005Metric_Pad0.72x0.64mm_HandSolder"
+		(property "Footprint" "Resistor_SMD:R_0805_2012Metric_Pad1.20x1.40mm_HandSolder"
 			(at 188.976 118.364 90)
 			(effects
@@
 			)
 		)
-		(property "Footprint" "Resistor_SMD:R_0402_1005Metric_Pad0.72x0.64mm_HandSolder"
+		(property "Footprint" "Resistor_SMD:R_0805_2012Metric_Pad1.20x1.40mm_HandSolder"
 			(at 98.806 137.414 90)
 			(effects
@@
 			)
 		)
-		(property "Footprint" "Resistor_SMD:R_0402_1005Metric_Pad0.72x0.64mm_HandSolder"
+		(property "Footprint" "Resistor_SMD:R_0805_2012Metric_Pad1.20x1.40mm_HandSolder"
 			(at 93.726 65.024 90)
 			(effects
@@
 			)
 		)
-		(property "Footprint" "Resistor_SMD:R_0402_1005Metric_Pad0.72x0.64mm_HandSolder"
+		(property "Footprint" "Resistor_SMD:R_0805_2012Metric_Pad1.20x1.40mm_HandSolder"
 			(at 121.666 137.414 90)
 			(effects
@@
 			)
 		)
-		(property "Footprint" "Resistor_SMD:R_0402_1005Metric_Pad0.72x0.64mm_HandSolder"
+		(property "Footprint" "Resistor_SMD:R_0805_2012Metric_Pad1.20x1.40mm_HandSolder"
 			(at 105.156 65.024 90)
 			(effects
@@
 			)
 		)
-		(property "Footprint" "Resistor_SMD:R_0402_1005Metric_Pad0.72x0.64mm_HandSolder"
+		(property "Footprint" "Resistor_SMD:R_0805_2012Metric_Pad1.20x1.40mm_HandSolder"
 			(at 61.214 120.904 90)
 			(effects

Commit message: wip
Parts:
- removed R1000, R1001: 0R, Resistor_SMD:R_0805_2012Metric_Pad1.20x1.40mm_HandSolder, symbol Device:R_US
Connections:
- net SC_RST: now also U6.3 (RSTIN)
- net at U6.10 (AUX1): now also J8.C4 (RFU)
Changed lines of the file:
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@@
 	(wire
 		(pts
-			(xy 181.61 91.44) (xy 210.82 91.44)
+			(xy 181.61 91.44) (xy 220.98 91.44)
 		)
 		(stroke
@@
 	(wire
 		(pts
-			(xy 115.57 101.6) (xy 118.11 101.6)
+			(xy 115.57 101.6) (xy 125.73 101.6)
 		)
 		(stroke
@@
 		(pts
 			(xy 53.34 88.9) (xy 92.71 88.9)
-		)
-		(stroke
-			(width 0)
-			(type default)
-		)
-	)
-	(wire
-		(pts
-			(xy 218.44 91.44) (xy 220.98 91.44)
 		)
 		(stroke
@@
 	)
 	(symbol
-		(lib_id "Device:R_US")
-		(at 214.63 91.44 90)
-		(unit 1)
-		(exclude_from_sim no)
-		(in_bom yes)
-		(on_board yes)
-		(dnp no)
-		(fields_autoplaced yes)
-		(property "Reference" "R1000"
-			(at 214.63 85.09 90)
-			(effects
-				(font
-					(size 1.27 1.27)
-				)
-			)
-		)
-		(property "Value" "0R"
-			(at 214.63 87.63 90)
-			(effects
-				(font
-					(size 1.27 1.27)
-				)
-			)
-		)
-		(property "Footprint" "Resistor_SMD:R_0805_2012Metric_Pad1.20x1.40mm_HandSolder"
-			(at 214.884 90.424 90)
-			(effects
-				(font
-					(size 1.27 1.27)
-				)
-				(hide yes)
-			)
-		)
-		(property "Datasheet" "~"
-			(at 214.63 91.44 0)
-			(effects
-				(font
-					(size 1.27 1.27)
-				)
-				(hide yes)
-			)
-		)
-		(property "Description" "Resistor, US symbol"
-			(at 214.63 91.44 0)
-			(effects
-				(font
-					(size 1.27 1.27)
-				)
-				(hide yes)
-			)
-		)
-		(pin "1"
-		)
-		(pin "2"
-		)
-		(instances
-			(project "Smartcard_Hat"
-				(path "/e63e39d7-6ac0-4ffd-8aa3-1841a4541b55/b93ee573-e5a5-4e8b-bced-8a93bd527c9a"
-					(reference "R1000")
-					(unit 1)
-				)
-			)
-		)
-	)
-	(symbol
 		(lib_id "Device:C")
 		(at 224.79 72.39 0)
@@
 					(unit 1)
 				)
-			)
-		)
-	)
-	(symbol
-		(lib_id "Device:R_US")
-		(at 121.92 101.6 90)
-		(unit 1)
-		(exclude_from_sim no)
-		(in_bom yes)
-		(on_board yes)
-		(dnp no)
-		(fields_autoplaced yes)
-		(property "Reference" "R1001"
-			(at 121.92 95.25 90)
-			(effects
-				(font
-					(size 1.27 1.27)
-				)
-			)
-		)
-		(property "Value" "0R"
-			(at 121.92 97.79 90)
-			(effects
-				(font
-					(size 1.27 1.27)
-				)
-			)
-		)
-		(property "Footprint" "Resistor_SMD:R_0805_2012Metric_Pad1.20x1.40mm_HandSolder"
-			(at 122.174 100.584 90)
-			(effects
-				(font
-					(size 1.27 1.27)
-				)
-				(hide yes)
-			)
-		)
-		(property "Datasheet" "~"
-			(at 121.92 101.6 0)
-			(effects
-				(font
-					(size 1.27 1.27)
-				)
-				(hide yes)
-			)
-		)
-		(property "Description" "Resistor, US symbol"
-			(at 121.92 101.6 0)
-			(effects
-				(font
-					(size 1.27 1.27)
-				)
-				(hide yes)
-			)
-		)
-		(pin "1"
-		)
-		(pin "2"
-		)
-		(instances
-			(project "Smartcard_Hat"
-				(path "/e63e39d7-6ac0-4ffd-8aa3-1841a4541b55/b93ee573-e5a5-4e8b-bced-8a93bd527c9a"
-					(reference "R1001")
-					(unit 1)
-				)
