File: shield/kicad/structure_diagram.kicad_sch (KiCad schematic)
At the start: 49 parts, among them J10 QR_FFC, J11 Arduino_D8-D13, J12 Arduino_D0-D7, J13 Arduino_Analog, J8 Smartcard, J9 Conn_01x08, U6 ST8034

Commit message: Add LCSC part numbers to all shield schematic components and verify pinouts
Added LCSC properties to 127 components across both schematic sheets:
- power.kicad_sch: 83 components (lib_symbols + instances)
- structure_diagram.kicad_sch: 44 components (lib_symbols + instances)

All IC pinouts verified against manufacturer datasheets:
- BQ25060DQCR (U1): 10-pin DFN, pins match TI datasheet
- TPS63060DSCR (U4): 10-pin VSON, pins match TI datasheet
- STC3100IST (U3): 8-pin DFN, pins match ST datasheet
- TPS3422EGDRYR (U2): 6-pin DFN, pins match TI datasheet
- MAX803SQ293D2T1G (U5): 3-pin SOT-23, pins match onsemi datasheet
- ST8034HNQR (U6): 24-pin QFN, pins match ST datasheet
- NTR4101PT1G (Q1,Q4): SOT-23 P-ch MOSFET, G/S/D verified
- DMG1012T (Q2,Q3,Q5,Q6): SOT-523 N-ch MOSFET, G/S/D verified

2 ICs not available on LCSC (TPS3422, MAX803) - noted for manual sourcing.
Updated README with comprehensive LCSC BOM table.

Agent-Logs-Url: https://github.com/3rdIteration/specter-diy/sessions/22e4313c-030b-4d7a-a876-9de4f55077cb

Co-authored-by: 3rdIteration <2230318+3rdIteration@users.noreply.github.com>
Parts:
- C29, C30, C31, C32, C33, C34, C38, C45, C48: LCSC (none) -> C1525
- C35, C36, C40, C42: LCSC (none) -> C784585
- C37, C41: LCSC (none) -> C307331
- C39: LCSC (none) -> C1560
- C43, C44, C46, C47: LCSC (none) -> C15850
- J10: LCSC (none) -> C88360
- LS1: LCSC (none) -> C76871
- R32, R33, R34, R35, R39, R43, R46, R47, R48, R49, R50, R52: LCSC (none) -> C25804
- R36, R40, R41, R42, R51: LCSC (none) -> C26083
- R37, R38: LCSC (none) -> C11702
- R44: LCSC (none) -> C25092
- R45: LCSC (none) -> C15000
- U6: LCSC (none) -> C2674058
Changed lines of the file:
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@@
+			(at 130 80 0)
+			(effects (font (size 1.27 1.27)) (hide yes)))
+		(property "LCSC" "C2674058"
 			(at 130 80 0)
 			(effects (font (size 1.27 1.27)) (hide yes)))
@@
 			(at 90 60 0)
 			(effects (font (size 1.27 1.27)) (hide yes)))
+		(property "LCSC" "C1525"
+			(at 90 60 0)
+			(effects (font (size 1.27 1.27)) (hide yes)))
 		(pin "1"
 )
@@
 			(at 90 72 0)
 			(effects (font (size 1.27 1.27)) (hide yes)))
+		(property "LCSC" "C1525"
+			(at 90 72 0)
+			(effects (font (size 1.27 1.27)) (hide yes)))
 		(pin "1"
 )
@@
 			(at 90 84 0)
 			(effects (font (size 1.27 1.27)) (hide yes)))
+		(property "LCSC" "C1525"
+			(at 90 84 0)
+			(effects (font (size 1.27 1.27)) (hide yes)))
 		(pin "1"
 )
@@
 			(at 90 96 0)
 			(effects (font (size 1.27 1.27)) (hide yes)))
+		(property "LCSC" "C1525"
+			(at 90 96 0)
+			(effects (font (size 1.27 1.27)) (hide yes)))
 		(pin "1"
 )
@@
 			(at 175 60 0)
 			(effects (font (size 1.27 1.27)) (hide yes)))
+		(property "LCSC" "C25804"
+			(at 175 60 0)
+			(effects (font (size 1.27 1.27)) (hide yes)))
 		(pin "1"
 )
@@
 			(at 175 72 0)
 			(effects (font (size 1.27 1.27)) (hide yes)))
+		(property "LCSC" "C25804"
+			(at 175 72 0)
+			(effects (font (size 1.27 1.27)) (hide yes)))
 		(pin "1"
 )
@@
 			(at 175 84 0)
 			(effects (font (size 1.27 1.27)) (hide yes)))
+		(property "LCSC" "C25804"
+			(at 175 84 0)
+			(effects (font (size 1.27 1.27)) (hide yes)))
 		(pin "1"
 )
@@
 			(at 175 96 0)
 			(effects (font (size 1.27 1.27)) (hide yes)))
+		(property "LCSC" "C25804"
+			(at 175 96 0)
+			(effects (font (size 1.27 1.27)) (hide yes)))
 		(pin "1"
 )
@@
 			(at 175 108 0)
 			(effects (font (size 1.27 1.27)) (hide yes)))
+		(property "LCSC" "C1525"
+			(at 175 108 0)
+			(effects (font (size 1.27 1.27)) (hide yes)))
 		(pin "1"
 )
@@
 			(effects (font (size 1.27 1.27)) (hide yes)))
 		(property "Datasheet" ""
+			(at 200 60 0)
+			(effects (font (size 1.27 1.27)) (hide yes)))
+		(property "LCSC" "C1525"
 			(at 200 60 0)
 			(effects (font (size 1.27 1.27)) (hide yes)))
@@
 			(at 80 165 0)
 			(effects (font (size 1.27 1.27)) (hide yes)))
+		(property "LCSC" "C88360"
+			(at 80 165 0)
+			(effects (font (size 1.27 1.27)) (hide yes)))
 		(pin "1"
 )
@@
 			(at 130 150 0)
 			(effects (font (size 1.27 1.27)) (hide yes)))
+		(property "LCSC" "C26083"
+			(at 130 150 0)
+			(effects (font (size 1.27 1.27)) (hide yes)))
 		(pin "1"
 )
@@
 			(at 130 162 0)
 			(effects (font (size 1.27 1.27)) (hide yes)))
+		(property "LCSC" "C11702"
+			(at 130 162 0)
+			(effects (font (size 1.27 1.27)) (hide yes)))
 		(pin "1"
 )
@@
 			(at 130 174 0)
 			(effects (font (size 1.27 1.27)) (hide yes)))
+		(property "LCSC" "C11702"
+			(at 130 174 0)
+			(effects (font (size 1.27 1.27)) (hide yes)))
 		(pin "1"
 )
@@
 			(at 55 155 0)
 			(effects (font (size 1.27 1.27)) (hide yes)))
+		(property "LCSC" "C784585"
+			(at 55 155 0)
+			(effects (font (size 1.27 1.27)) (hide yes)))
 		(pin "1"
 )
@@
 			(effects (font (size 1.27 1.27)) (hide yes)))
 		(property "Datasheet" ""
+			(at 55 170 0)
+			(effects (font (size 1.27 1.27)) (hide yes)))
+		(property "LCSC" "C784585"
 			(at 55 170 0)
 			(effects (font (size 1.27 1.27)) (hide yes)))
@@
 			(at 70 240 0)
 			(effects (font (size 1.27 1.27)) (hide yes)))
+		(property "LCSC" "C76871"
+			(at 70 240 0)
+			(effects (font (size 1.27 1.27)) (hide yes)))
 		(pin "1"
 )
@@
 			(effects (font (size 1.27 1.27)) (hide yes)))
 		(property "Datasheet" ""
+			(at 45 235 0)
+			(effects (font (size 1.27 1.27)) (hide yes)))
+		(property "LCSC" "C25804"
 			(at 45 235 0)
 			(effects (font (size 1.27 1.27)) (hide yes)))
@@
 			(at 40 295 0)
 			(effects (font (size 1.27 1.27)) (hide yes)))
+		(property "LCSC" "C26083"
+			(at 40 295 0)
+			(effects (font (size 1.27 1.27)) (hide yes)))
 		(pin "1"
 )
@@
 			(at 62 295 0)
 			(effects (font (size 1.27 1.27)) (hide yes)))
+		(property "LCSC" "C26083"
+			(at 62 295 0)
+			(effects (font (size 1.27 1.27)) (hide yes)))
 		(pin "1"
 )
@@
 			(at 84 295 0)
 			(effects (font (size 1.27 1.27)) (hide yes)))
+		(property "LCSC" "C26083"
+			(at 84 295 0)
+			(effects (font (size 1.27 1.27)) (hide yes)))
 		(pin "1"
 )
@@
 			(at 106 295 0)
 			(effects (font (size 1.27 1.27)) (hide yes)))
+		(property "LCSC" "C25804"
+			(at 106 295 0)
+			(effects (font (size 1.27 1.27)) (hide yes)))
 		(pin "1"
 )
@@
 			(at 128 295 0)
 			(effects (font (size 1.27 1.27)) (hide yes)))
+		(property "LCSC" "C25092"
+			(at 128 295 0)
+			(effects (font (size 1.27 1.27)) (hide yes)))
 		(pin "1"
 )
@@
 			(at 150 295 0)
 			(effects (font (size 1.27 1.27)) (hide yes)))
+		(property "LCSC" "C15000"
+			(at 150 295 0)
+			(effects (font (size 1.27 1.27)) (hide yes)))
 		(pin "1"
 )
@@
 			(at 172 295 0)
 			(effects (font (size 1.27 1.27)) (hide yes)))
+		(property "LCSC" "C25804"
+			(at 172 295 0)
+			(effects (font (size 1.27 1.27)) (hide yes)))
 		(pin "1"
 )
@@
 			(at 194 295 0)
 			(effects (font (size 1.27 1.27)) (hide yes)))
+		(property "LCSC" "C25804"
+			(at 194 295 0)
+			(effects (font (size 1.27 1.27)) (hide yes)))
 		(pin "1"
 )
@@
 			(at 216 295 0)
 			(effects (font (size 1.27 1.27)) (hide yes)))
+		(property "LCSC" "C25804"
+			(at 216 295 0)
+			(effects (font (size 1.27 1.27)) (hide yes)))
 		(pin "1"
 )
@@
 			(at 238 295 0)
 			(effects (font (size 1.27 1.27)) (hide yes)))
+		(property "LCSC" "C25804"
+			(at 238 295 0)
+			(effects (font (size 1.27 1.27)) (hide yes)))
 		(pin "1"
 )
@@
 			(at 260 295 0)
 			(effects (font (size 1.27 1.27)) (hide yes)))
+		(property "LCSC" "C25804"
+			(at 260 295 0)
+			(effects (font (size 1.27 1.27)) (hide yes)))
 		(pin "1"
 )
@@
 			(at 282 295 0)
 			(effects (font (size 1.27 1.27)) (hide yes)))
+		(property "LCSC" "C26083"
+			(at 282 295 0)
+			(effects (font (size 1.27 1.27)) (hide yes)))
 		(pin "1"
 )
@@
 			(at 304 295 0)
 			(effects (font (size 1.27 1.27)) (hide yes)))
+		(property "LCSC" "C25804"
+			(at 304 295 0)
+			(effects (font (size 1.27 1.27)) (hide yes)))
 		(pin "1"
 )
@@
 			(at 326 295 0)
 			(effects (font (size 1.27 1.27)) (hide yes)))
+		(property "LCSC" "C307331"
+			(at 326 295 0)
+			(effects (font (size 1.27 1.27)) (hide yes)))
 		(pin "1"
 )
@@
 			(at 348 295 0)
 			(effects (font (size 1.27 1.27)) (hide yes)))
+		(property "LCSC" "C1525"
+			(at 348 295 0)
+			(effects (font (size 1.27 1.27)) (hide yes)))
 		(pin "1"
 )
@@
 			(at 370 295 0)
 			(effects (font (size 1.27 1.27)) (hide yes)))
+		(property "LCSC" "C1560"
+			(at 370 295 0)
+			(effects (font (size 1.27 1.27)) (hide yes)))
 		(pin "1"
 )
@@
 			(at 40 317 0)
 			(effects (font (size 1.27 1.27)) (hide yes)))
+		(property "LCSC" "C784585"
+			(at 40 317 0)
+			(effects (font (size 1.27 1.27)) (hide yes)))
 		(pin "1"
 )
@@
 			(at 62 317 0)
 			(effects (font (size 1.27 1.27)) (hide yes)))
+		(property "LCSC" "C307331"
+			(at 62 317 0)
+			(effects (font (size 1.27 1.27)) (hide yes)))
 		(pin "1"
 )
@@
 			(at 84 317 0)
 			(effects (font (size 1.27 1.27)) (hide yes)))
+		(property "LCSC" "C784585"
+			(at 84 317 0)
+			(effects (font (size 1.27 1.27)) (hide yes)))
 		(pin "1"
 )
@@
 			(at 106 317 0)
 			(effects (font (size 1.27 1.27)) (hide yes)))
+		(property "LCSC" "C15850"
+			(at 106 317 0)
+			(effects (font (size 1.27 1.27)) (hide yes)))
 		(pin "1"
 )
@@
 			(at 128 317 0)
 			(effects (font (size 1.27 1.27)) (hide yes)))
+		(property "LCSC" "C15850"
+			(at 128 317 0)
+			(effects (font (size 1.27 1.27)) (hide yes)))
 		(pin "1"
 )
@@
 			(at 150 317 0)
 			(effects (font (size 1.27 1.27)) (hide yes)))
+		(property "LCSC" "C1525"
+			(at 150 317 0)
+			(effects (font (size 1.27 1.27)) (hide yes)))
 		(pin "1"
 )
@@
 			(at 172 317 0)
 			(effects (font (size 1.27 1.27)) (hide yes)))
+		(property "LCSC" "C15850"
+			(at 172 317 0)
+			(effects (font (size 1.27 1.27)) (hide yes)))
 		(pin "1"
 )
@@
 			(at 194 317 0)
 			(effects (font (size 1.27 1.27)) (hide yes)))
+		(property "LCSC" "C15850"
+			(at 194 317 0)
+			(effects (font (size 1.27 1.27)) (hide yes)))
 		(pin "1"
 )
@@
 			(at 216 317 0)
 			(effects (font (size 1.27 1.27)) (hide yes)))
+		(property "LCSC" "C1525"
+			(at 216 317 0)
+			(effects (font (size 1.27 1.27)) (hide yes)))
